File: v2.0/USB/USB_conn.kicad_pcb (KiCad board)
At the start: 2 copper layers, 21.8 x 20.5 mm, 11 parts, among them J1 Conn_01x10, J10 Conn_01x01, J11 Conn_01x01, J2 Conn_01x01, J3 Conn_01x01, J4 Conn_01x01, J5 Conn_01x01, J6 Conn_01x01, J7 Conn_01x01, J8 Conn_01x01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

Commit message: updated files
Connections:
- J1 pad 1: SW2 -> SDA
- J1 pad 2: SW1 -> SCL
- J1 pad 3: +3V3 -> SW2
- J1 pad 4: INT_N -> USB_N
- J1 pad 5: SDA -> USB_P
- J1 pad 6: SCL -> +3V3
- J1 pad 7: USB_N -> SW1
- J1 pad 8: USB_P -> INT_N
Routing:
- net +3V3: track 15.5 -> 30.9 mm, vias 0 -> 1
- net SW1: track 15.3 -> 30.2 mm, vias 0 -> 1
- net INT_N: track 17.8 -> 29.0 mm, vias 0 -> 1
- net SW2: track 15.1 -> 21.6 mm
- net USB_N: track 18.2 -> 20.8 mm
- net USB_P: track 17.2 -> 19.8 mm
- net SCL: track 21.9 -> 19.7 mm, vias 1 -> 0
Other:
- rule trace_min: 0.2 -> 0.127
